File: Simulaciones/KiCAD/Inversor/Inversor.kicad_pcb (KiCad board)
At the start: 2 copper layers, 8 parts, among them J1 In, J2 Out, J3 GND, J4 Vcc, U1 LM358

Commit message: Otro PCB. quién carajo me mandó a meterme acá
Routing:
- net GND: track 84.3 -> 86.8 mm
Other:
- board outline added: 65 x 50 mm
Changed lines of the file:
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@@
 		)
 	)
+	(gr_rect
+		(start 140 80)
+		(end 205 130)
+		(stroke
+			(width 0.05)
+			(type default)
+		)
+		(fill no)
+		(layer "Edge.Cuts")
+	)
 	(segment
-		(start 144.25 92)
-		(end 153.19 92)
+		(start 150.31 121.56)
+		(end 150 121.25)
 		(width 0.2)
 		(layer "F.Cu")
-		(net "Net-(J1-Pin_1)")
+		(net "GND")
+	)
+	(segment
+		(start 150 101)
+		(end 168.605 101)
+		(width 0.2)
+		(layer "F.Cu")
+		(net "GND")
+	)
+	(segment
+		(start 168.605 101)
+		(end 168.63 101.025)
+		(width 0.2)
+		(layer "F.Cu")
+		(net "GND")
+	)
+	(segment
+		(start 189.5 121.56)
+		(end 150.31 121.56)
+		(width 0.2)
+		(layer "F.Cu")
+		(net "GND")
+	)
+	(segment
+		(start 171.17 101.025)
+		(end 168.63 101.025)
+		(width 0.2)
+		(layer "F.Cu")
+		(net "GND")
+	)
+	(segment
+		(start 150 121.25)
+		(end 150 101)
+		(width 0.2)
+		(layer "F.Cu")
+		(net "GND")
+	)
+	(segment
+		(start 144.25 101)
+		(end 150 101)
+		(width 0.2)
+		(layer "F.Cu")
+		(net "GND")
 	)
 	(segment
@@
 	)
 	(segment
-		(start 150.31 121.56)
-		(end 150 121.25)
+		(start 144.25 92)
+		(end 153.19 92)
 		(width 0.2)
 		(layer "F.Cu")
-		(net "GND")
-	)
-	(segment
-		(start 150 101)
-		(end 168.605 101)
-		(width 0.2)
-		(layer "F.Cu")
-		(net "GND")
-	)
-	(segment
-		(start 168.605 101)
-		(end 168.63 101.025)
-		(width 0.2)
-		(layer "F.Cu")
-		(net "GND")
-	)
-	(segment
-		(start 189.5 121.56)
-		(end 150.31 121.56)
-		(width 0.2)
-		(layer "F.Cu")
-		(net "GND")
-	)
-	(segment
-		(start 150 121.25)
-		(end 150 101)
-		(width 0.2)
-		(layer "F.Cu")
-		(net "GND")
-	)
-	(segment
-		(start 144.25 101)
-		(end 150 101)
-		(width 0.2)
-		(layer "F.Cu")
-		(net "GND")
-	)
-	(segment
-		(start 176.25 108.645)
-		(end 176.25 115)
-		(width 0.2)
-		(layer "F.Cu")
-		(net "Net-(J4-Pin_1)")
+		(net "Net-(J1-Pin_1)")
 	)
 	(segment
@@
 		(net "Net-(U1A--)")
 	)
+	(segment
+		(start 176.25 108.645)
+		(end 176.25 115)
+		(width 0.2)
+		(layer "F.Cu")
+		(net "Net-(J4-Pin_1)")
+	)
 	(embedded_fonts no)
